File: _autosave-mutebox_hat_audio_in.kicad_pcb (KiCad board)
At the start: 2 copper layers, 65 x 56 mm, 43 parts, among them J1 GPIO, J2 PLR237/T10BK, U1 CAT24C256, U2 74LVC157, U3 PCM1862DBT, U4 DIR9001PW, Y1 12.288 MHz, Y3 XO32

Commit message: More fixes
Connections:
- C10 pad 1: 3V3_A -> /VREF
- C10 pad 2: Net-(U3-VREF) -> GND
- C12 pad 1: 3V3_A -> /VREF
- C12 pad 2: Net-(U3-VREF) -> GND
- J_L_IN1 pad 2: 3V3_A -> /VREF
- J_R_IN1 pad 2: 3V3_A -> /VREF
- U3 pad 1: 3V3_A -> /VREF
- U3 pad 2: 3V3_A -> /VREF
- U3 pad 6: Net-(U3-VREF) -> /VREF
- U3 pad 7: 3V3_A -> GND
- Y3 pad 1: 3V3_A -> GND
- Y3 pad 2: 3V3_A -> GND
- Y3 pad 4: 3V3_A -> GND
Routing:
- net GND: track 65.0 -> 76.1 mm, vias 15 -> 17
- net Net-(U3-VREF): track 11.2 -> 0.00 mm, vias 2 -> 0
