File: _autosave-mutebox_hat_audio_in.kicad_pcb (KiCad board)
At the start: 2 copper layers, 65 x 56 mm, 56 parts, among them J1 GPIO, J2 PLR237/T10BK, J3 RCJ-042, J4 RCJ-042, U2 74LVC157, U3 PCM1862DBT, U5 DIR9001PW, Y3 XO32

Commit message: Final changes before ordering.
Parts:
- D3, D4: value LED -> NCD0805R1
